File: arduino-shield/arduino-shield.kicad_sch (KiCad schematic)
At the start: 15 parts, among them J1 393800102, J2 393800102, J3 393800102, Q1 TIP120, Q2 TIP120, SW1 100SP4T1B2M2QE, SW2 100SP4T1B2M2QE, SW3 ANT13SECQE

Commit message: Expand BOM and assembly docs; add shield placement image.
Document DigiKey line items, step-by-step assembly with arduino-shield.jpg,
nylon M3 mounting for Q1/Q2, and updated shield Gerbers/KiCad exports.

Co-authored-by: Cursor <cursoragent@cursor.com>
Parts:
- renumbered D2 to D1, D3 to D2, D1 to D3, J2 to J1, J3 to J2, J1 to J3, Q2 to Q1, Q1 to Q2, SW3 to SW1, SW1 to SW2, SW2 to SW3, TDK_PS1240P02BT to TDK_PS1240P02BT1
Connections:
- net 12vdc: now also J2.2 (Pin_2); no longer J2.1 (Pin_1)
- net GND: now also J2.1 (Pin_1); no longer J2.2 (Pin_2)
